File: PCB/spark.kicad_sch (KiCad schematic)
At the start: 41 parts, among them J1 JST connector, J2 Conn_01x04, SW1 SW_Push_45deg, SW10 SW_Push_45deg, SW11 SW_Push_45deg, SW12 SW_Push_45deg, SW13 SW_Push_45deg, SW14 SW_Push_45deg, SW15 SW_Push_45deg, SW16 SW_Push_45deg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

Commit message: Routed everything
Parts:
- removed J2: Conn_01x04, symbol Connector_Generic:Conn_01x04
- removed U1: SuperMini nRF52840, KiCAD_Stuff:ProMicro_jumpable, symbol PCM_marbastlib-promicroish:SuperMini_nRF52840
- added U1: Nice_Nano_V2, ScottoKeebs_MCU:Nice_Nano_V2, symbol ScottoKeebs:MCU_Nice_Nano_V2
- D1, D10, D11, D12, D13, D14, D15, D16, D17, D18, D2, D3, D4, D5, D6, D7, D8, D9: footprint Diode_THT:D_DO-35_SOD27_P7.62mm_Horizontal -> KiCAD_Stuff:1N4148 Cutout Diode
- J1: footprint (none) -> KiCAD_Stuff:Connector_1x02_JST-PH
- SW19: footprint (none) -> KiCAD_Stuff:SW_SPST_B3U-1000P_Reversible
- SW20: footprint PCM_marbastlib-various:SW_MSK12C02-HB -> PCM_marbastlib-various:SW_MSK12C02-HB_Reversible
Connections:
- net Bat+: now also U1.24 (B+)
- net Col1: now also U1.5 (2)
- net Col2: now also U1.6 (3)
- net Col3: now also U1.7 (4)
- net Col4: now also U1.8 (5)
- net Col5: now also U1.9 (6)
- net GND: now also U1.23 (GND), U1.3 (GND), U1.4 (GND)
- net Reset: now also U1.22 (RST)
- net Row1: now also U1.2 (0)
- net Row2: now also U1.10 (7)
- net Row3: now also U1.11 (8)
- net Row4: now also U1.12 (9)
- no-connect marks 2 -> 12
